File: ArudinoShield.sch (EAGLE design)
At the start: 24 parts, among them IC1 L298

Commit message: updated schematic and board
Parts:
- added 9G: (no value), pinhead:PINHD-1X3
- renumbered IN1 to VIN
Connections:
- net N$1 renamed ENA
- net N$15 renamed OUT1
- net N$16 renamed OUT2
- net N$17 renamed OUT3
- net N$18 renamed OUT4
- net N$2 renamed IN3
- net N$20 renamed ENB
- net N$21 renamed IN1
- net N$22 renamed IN2
- net N$24 renamed IN4
- net N$31 renamed VIN
- net N$7 renamed ECHO
- net N$8 renamed TRIG
- removed net N$26: B1.VIN, C2.1, IC1.VCC, R3.2, VREG.VOUT
- removed net N$29: B1.GND@1, C1.2, C2.2, D5.A, D6.A, D7.A, D8.A, IC1.GND, IC1.SEN_A, LED1.C, OUT1.2, OUT2.2, OUT3.2, OUT4.2, VIN.1, VREG.GND
- removed net N$9: B1.GND@2, HC-SR04.4
- new net +5V: 9G.2, B1.VIN, C2.1, IC1.VCC, R3.2, VREG.VOUT
- new net 9GPWM: 9G.1, B1.*D11
- new net GND: 9G.3, B1.GND@1, C1.2, C2.2, D5.A, D6.A, D7.A, D8.A, HC-SR04.4, IC1.GND, IC1.SEN_A, IC1.SEN_B, LED1.C, OUT1.2, OUT2.2, OUT3.2, OUT4.2, VIN.1, VREG.GND
Other:
- moved on the sheet: R2

Commit message: updated power trace size
Parts:
- removed HC-05: (no value), pinhead:PINHD-1X4
- added HC05: (no value), pinhead:PINHD-1X6/90
Connections:
- removed net N$10: B1.5V, HC-05.1, HC-SR04.1
- net +5V: now also B1.5V, HC-SR04.1, HC05.2
- net N$12: now also HC05.4; no longer HC-05.3
- net N$13: now also HC05.3; no longer HC-05.2
- net N$14: now also HC05.5; no longer HC-05.4
Changed lines of the file:
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@@
 <part name="B1" library="SparkFun-Boards" library_urn="urn:adsk.eagle:library:509" deviceset="ARDUINO_UNO_R3_SHIELD" device="BASIC" package3d_urn="urn:adsk.eagle:package:37321/1"/>
 <part name="HC-SR04" library="pinhead" library_urn="urn:adsk.eagle:library:325" deviceset="PINHD-1X4" device="" package3d_urn="urn:adsk.eagle:package:22407/2"/>
-<part name="HC-05" library="pinhead" library_urn="urn:adsk.eagle:library:325" deviceset="PINHD-1X4" device="" package3d_urn="urn:adsk.eagle:package:22407/2"/>
 <part name="R1" library="adafruit" deviceset="R-US_" device="0207/7" value="1k"/>
 <part name="R2" library="adafruit" deviceset="R-US_" device="0207/7" value="2K"/>
@@
 <part name="OUT4" library="con-amp" library_urn="urn:adsk.eagle:library:127" deviceset="MTA02-156" device="" package3d_urn="urn:adsk.eagle:package:8081562/1"/>
 <part name="9G" library="pinhead" library_urn="urn:adsk.eagle:library:325" deviceset="PINHD-1X3" device="" package3d_urn="urn:adsk.eagle:package:22458/2"/>
+<part name="HC05" library="pinhead" library_urn="urn:adsk.eagle:library:325" deviceset="PINHD-1X6" device="/90" package3d_urn="urn:adsk.eagle:package:22475/2"/>
 </parts>
 <sheets>
@@
 <attribute name="VALUE" x="24.13" y="68.58" size="1.778" layer="96" rot="R180"/>
 </instance>
-<instance part="HC-05" gate="A" x="104.14" y="71.12" smashed="yes">
-<attribute name="NAME" x="97.79" y="79.375" size="1.778" layer="95"/>
-<attribute name="VALUE" x="97.79" y="63.5" size="1.778" layer="96"/>
-</instance>
 <instance part="R1" gate="G$1" x="91.44" y="68.58" smashed="yes">
 <attribute name="NAME" x="87.63" y="70.0786" size="1.778" layer="95"/>
@@
 <attribute name="NAME" x="24.13" y="22.225" size="1.778" layer="95" rot="R180"/>
 <attribute name="VALUE" x="24.13" y="35.56" size="1.778" layer="96" rot="R180"/>
+</instance>
+<instance part="HC05" gate="A" x="116.84" y="71.12" smashed="yes">
+<attribute name="NAME" x="110.49" y="81.915" size="1.778" layer="95"/>
+<attribute name="VALUE" x="110.49" y="60.96" size="1.778" layer="96"/>
 </instance>
 </instances>
@@
 </segment>
 </net>
-<net name="N$10" class="0">
-<segment>
-<pinref part="B1" gate="G$1" pin="5V"/>
-<wire x1="50.8" y1="43.18" x2="45.72" y2="43.18" width="0.1524" layer="91"/>
-<wire x1="45.72" y1="43.18" x2="25.4" y2="43.18" width="0.1524" layer="91"/>
-<wire x1="25.4" y1="43.18" x2="25.4" y2="55.88" width="0.1524" layer="91"/>
-<pinref part="HC-05" gate="A" pin="1"/>
-<wire x1="101.6" y1="76.2" x2="45.72" y2="76.2" width="0.1524" layer="91"/>
-<wire x1="45.72" y1="76.2" x2="45.72" y2="43.18" width="0.1524" layer="91"/>
-<junction x="45.72" y="43.18"/>
-<pinref part="HC-SR04" gate="A" pin="1"/>
-<wire x1="25.4" y1="55.88" x2="20.32" y2="55.88" width="0.1524" layer="91"/>
-</segment>
-</net>
 <net name="N$12" class="0">
 <segment>
-<pinref part="HC-05" gate="A" pin="3"/>
-<wire x1="101.6" y1="71.12" x2="76.2" y2="71.12" width="0.1524" layer="91"/>
+<wire x1="114.3" y1="71.12" x2="76.2" y2="71.12" width="0.1524" layer="91"/>
 <pinref part="B1" gate="G$1" pin="RX"/>
+<pinref part="HC05" gate="A" pin="4"/>
 </segment>
 </net>
 <net name="N$13" class="0">
 <segment>
-<pinref part="HC-05" gate="A" pin="2"/>
-<wire x1="101.6" y1="73.66" x2="91.44" y2="73.66" width="0.1524" layer="91"/>
-<wire x1="91.44" y1="73.66" x2="91.44" y2="81.28" width="0.1524" layer="91"/>
-<wire x1="91.44" y1="81.28" x2="109.22" y2="81.28" width="0.1524" layer="91"/>
-<wire x1="109.22" y1="81.28" x2="109.22" y2="17.78" width="0.1524" layer="91"/>
+<wire x1="109.22" y1="73.66" x2="109.22" y2="17.78" width="0.1524" layer="91"/>
 <wire x1="109.22" y1="17.78" x2="83.82" y2="17.78" width="0.1524" layer="91"/>
 <pinref part="B1" gate="G$1" pin="GND@0"/>
@@
 <wire x1="83.82" y1="27.94" x2="83.82" y2="17.78" width="0.1524" layer="91"/>
 <junction x="83.82" y="17.78"/>
+<pinref part="HC05" gate="A" pin="3"/>
+<wire x1="114.3" y1="73.66" x2="109.22" y2="73.66" width="0.1524" layer="91"/>
 </segment>
 </net>
@@
 <segment>
 <pinref part="R1" gate="G$1" pin="2"/>
-<pinref part="HC-05" gate="A" pin="4"/>
-<wire x1="96.52" y1="68.58" x2="101.6" y2="68.58" width="0.1524" layer="91"/>
+<wire x1="96.52" y1="68.58" x2="114.3" y2="68.58" width="0.1524" layer="91"/>
+<pinref part="HC05" gate="A" pin="5"/>
 </segment>
 </net>
@@
 <junction x="38.1" y="27.94"/>
 </segment>
-</net>
+<segment>
+<pinref part="B1" gate="G$1" pin="5V"/>
+<wire x1="50.8" y1="43.18" x2="45.72" y2="43.18" width="0.1524" layer="91"/>
+<wire x1="45.72" y1="43.18" x2="25.4" y2="43.18" width="0.1524" layer="91"/>
+<wire x1="25.4" y1="43.18" x2="25.4" y2="55.88" width="0.1524" layer="91"/>
+<wire x1="114.3" y1="76.2" x2="45.72" y2="76.2" width="0.1524" layer="91"/>
+<wire x1="45.72" y1="76.2" x2="45.72" y2="43.18" width="0.1524" layer="91"/>
+<junction x="45.72" y="43.18"/>
+<pinref part="HC-SR04" gate="A" pin="1"/>
+<wire x1="25.4" y1="55.88" x2="20.32" y2="55.88" width="0.1524" layer="91"/>
+<label x="30.48" y="43.18" size="1.6764" layer="95"/>
+<pinref part="HC05" gate="A" pin="2"/>
+</segment>
+</net>
