File: EAGLE/ATMegaBoard.sch (EAGLE design)
At the start: 30 parts, among them IC1 L298, IC2 ATMEGA168-20P, IC3 REG1117, X1 49S/18PF

Commit message: set EN on HC-05 to +5v
Connections:
- net +5V: now also HC05.1
Changed lines of the file:
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@@
 <wire x1="101.6" y1="-12.7" x2="96.52" y2="-12.7" width="0.1524" layer="91"/>
 <label x="96.52" y="-12.7" size="1.778" layer="95"/>
+<pinref part="HC05" gate="G$1" pin="1"/>
+<wire x1="101.6" y1="-10.16" x2="101.6" y2="-12.7" width="0.1524" layer="91"/>
+<junction x="101.6" y="-12.7"/>
 </segment>
 <segment>
